File: vco/pcb/vco.kicad_pcb (KiCad board)
At the start: 2 copper layers, 50.5 x 108.5 mm, 98 parts, among them J1 Conn_02x05_Odd_Even, J10 AudioJack2_SwitchT, J2 AudioJack2_SwitchT, J3 AudioJack2_SwitchT, J4 AudioJack2_SwitchT, J5 AudioJack2_SwitchT, J6 AudioJack2_SwitchT, J7 AudioJack2_SwitchT, J8 AudioJack2_SwitchT, J9 AudioJack2_SwitchT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

Commit message: vco: Generate production files for the PCB
Other:
- board text added: "JLCJLCJLCJLC"
Changed lines of the file:
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@@
       (layerselection 0x00010fc_ffffffff)
       (disableapertmacros false)
-      (usegerberextensions false)
-      (usegerberattributes true)
-      (usegerberadvancedattributes true)
-      (creategerberjobfile true)
+      (usegerberextensions true)
+      (usegerberattributes false)
+      (usegerberadvancedattributes false)
+      (creategerberjobfile false)
       (svguseinch false)
       (svgprecision 6)
@@
       (plotinvisibletext false)
       (sketchpadsonfab false)
-      (subtractmaskfromsilk false)
+      (subtractmaskfromsilk true)
       (outputformat 1)
       (mirror false)
-      (drillshape 1)
+      (drillshape 0)
       (scaleselection 1)
-      (outputdirectory "")
+      (outputdirectory "gerber")
     )
   )
@@
     (effects (font (size 1 1) (thickness 0.2)))
   )
+  (gr_text "JLCJLCJLCJLC" (at 140.335 156.21) (layer "F.SilkS")
+    (effects (font (size 1.2 1.2) (thickness 0.3)))
+  )
   (gr_text "Activity LED" (at 155.321 56.388) (layer "F.SilkS")
     (effects (font (size 1 1) (thickness 0.2)))
@@
     (style (thickness 0.2) (arrow_length 1.27) (text_position_mode 0) (extension_height 0.58642) (extension_offset 0.5) keep_text_aligned)
   )
-  (dimension (type orthogonal) (layer "F.Cu")
-    (pts (xy 165.608 51.486295) (xy 162.348 54.864))
-    (height 2.794)
-    (orientation 1)
-    (gr_text "3.3777 mm" (at 166.602 53.175147 90) (layer "F.Cu")
-      (effects (font (size 1.5 1.5) (thickness 0.3)))
-    )
-    (format (units 3) (units_format 1) (precision 4))
-    (style (thickness 0.2) (arrow_length 1.27) (text_position_mode 0) (extension_height 0.58642) (extension_offset 0.5) keep_text_aligned)
-  )
   (dimension (type orthogonal) (layer "Dwgs.User")
     (pts (xy 160.358 112.156295) (xy 152.823 129.656295))
@@
       (effects (font (size 1.5 1.5) (thickness 0.3)))
     )
+    (format (units 3) (units_format 1) (precision 4))
+    (style (thickness 0.2) (arrow_length 1.27) (text_position_mode 0) (extension_height 0.58642) (extension_offset 0.5) keep_text_aligned)
+  )
+  (dimension (type orthogonal) (layer "Dwgs.User")
+    (pts (xy 165.608 51.486295) (xy 162.348 54.864))
+    (height 2.794)
+    (orientation 1)
+    (gr_text "3.3777 mm" (at 166.602 53.175147 90) (layer "Dwgs.User")
+      (effects (font (size 1.5 1.5) (thickness 0.3)))
+    )

Commit message: vco: Small update
Parts:
- moved D2 2.79 mm to (128.8, 56.9)
- moved C3 2.79 mm to (129.2, 61.2)
- moved C4 2.79 mm to (129.2, 59.7)
- moved D1 2.79 mm to (128.8, 64.0)
- moved C1 2.79 mm to (133.3, 61.2)
- moved C2 2.79 mm to (133.3, 59.7)
- moved J1 2.23 mm to (121.6, 55.4)
Connections:
- J2 pad TN: GND -> unconnected-(J2-PadTN)
- J3 pad TN: GND -> unconnected-(J3-PadTN)
- J7 pad TN: GND -> unconnected-(J7-PadTN)
- J8 pad TN: GND -> unconnected-(J8-PadTN)
Routing:
- net +12V: track 245.1 -> 240.8 mm
- net -12V: track 221.7 -> 217.8 mm, vias 13 -> 12
Other:
- board text added: "+12V"
- board text added: "-12V"
