File: vco/pcb/vco.kicad_sch (KiCad schematic)
At the start: 0 parts

Commit message: vco: Update headers in pcb
Other:
- company: (none) -> L. Rittel
Changed lines of the file:
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@@
   (title_block
     (title "Eurorack VCO")
-    (date "2022-12-30")
-    (rev "Rev. 1")
+    (date "2022-12-31")
+    (rev "Rev. 1 2022")
+    (company "L. Rittel")
   )
   (sheet (at 88.9 27.94) (size 55.88 45.72) (fields_autoplaced)
