File: breadboard-breakout/breadboard-breakout.kicad_pcb (KiCad board)
At the start: 2 copper layers, 40 x 108.5 mm, 35 parts, among them J1 Conn_02x05_Odd_Even, J10 AudioJack2_SwitchT, J11 AudioJack2_SwitchT, J12 Conn_02x03_Odd_Even, J13 Conn_01x02, J14 Conn_01x02, J15 Conn_01x02, J16 Conn_01x02, J2 Conn_01x03, J3 Conn_01x03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

Commit message: breakout: Finish the PCB
Parts:
- removed G***: LOGO, LOGO
Routing:
- net Net-(J6-Pad2): track 19.4 -> 24.6 mm
- net Net-(J6-Pad1): track 18.9 -> 23.7 mm
- net Net-(J3-Pad1): track 67.2 -> 71.6 mm
- net Net-(J8-PadTN): track 128.4 -> 132.0 mm, vias 2 -> 4
- net Net-(J3-Pad3): track 72.8 -> 75.6 mm
- net Net-(R1-Pad2): track 119.8 -> 122.4 mm, vias 2 -> 4
- net Net-(RV2-Pad2): track 70.8 -> 73.1 mm
- net Net-(J5-Pad1): track 48.8 -> 51.1 mm
- net Net-(J5-Pad2): track 51.6 -> 53.4 mm
- net Net-(J5-Pad3): track 52.8 -> 54.6 mm
- net Net-(R4-Pad2): track 46.1 -> 47.8 mm
- net Net-(J4-Pad1): track 45.4 -> 47.0 mm
- net Net-(RV3-Pad2): track 49.0 -> 50.6 mm
- net Net-(J4-Pad3): track 52.6 -> 54.1 mm
- net Net-(J7-Pad3): track 23.7 -> 25.1 mm
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Other:
- board text added: "Escape Rev.1 2023 L. Rittel"
- board text added: "JLCJLCJLCJLC"

Commit message: breakout: finalize the pcb
Parts:
- J1: footprint Connector_PinSocket_2.54mm:PinSocket_2x05_P2.54mm_Vertical -> Connector_PinHeader_2.54mm:PinHeader_2x05_P2.54mm_Vertical
- moved J1 2.56 mm to (-6.35, -39.4)
