File: breadboard-breakout/breadboard-breakout.kicad_sch (KiCad schematic)
At the start: 29 parts

Commit message: breakout: WIP
Parts:
- removed C? (x2): 10u, symbol Device:C_Polarized
- removed J? (x3): Conn_01x03, symbol Connector_Generic:Conn_01x03
- removed J?: Conn_01x04, symbol Connector_Generic:Conn_01x04
- removed RV? (x2): R_Potentiometer, symbol Device:R_Potentiometer
- added C1, C2: 10u, Capacitor_SMD:C_0603_1608Metric_Pad1.08x0.95mm_HandSolder, symbol Device:C
- added J12: Conn_02x03_Odd_Even, Connector_PinSocket_2.54mm:PinSocket_2x03_P2.54mm_Vertical, symbol Connector_Generic:Conn_02x03_Odd_Even
- added J13, J14, J15, J16: Conn_01x02, Connector_PinSocket_2.54mm:PinSocket_1x02_P2.54mm_Vertical, symbol Connector_Generic:Conn_01x02
- added J3, J4, J5: Conn_01x03, Connector_PinSocket_2.54mm:PinSocket_1x03_P2.54mm_Vertical, symbol Connector_Generic:Conn_01x03
- added RV2, RV3, RV4: 10k, Potentiometer_THT:Potentiometer_Alpha_RD901F-40-00D_Single_Vertical, symbol Device:R_Potentiometer
- C3, C4: renamed from C?; footprint (none) -> Capacitor_SMD:C_0603_1608Metric_Pad1.08x0.95mm_HandSolder
- D1, D2: renamed from D?; value D -> B130-13F; footprint (none) -> Diode_SMD:D_SMA_Handsoldering
- F1, F2: renamed from F?; value Fuse -> Fuse 1206; footprint (none) -> Fuse:Fuse_1206_3216Metric_Pad1.42x1.75mm_HandSolder
- J1: renamed from J?; footprint (none) -> Connector_PinSocket_2.54mm:PinSocket_2x05_P2.54mm_Vertical
- J10, J11, J8, J9: renamed from J?; footprint (none) -> Connector_Audio:Jack_3.5mm_QingPu_WQP-PJ398SM_Vertical_CircularHoles
- J2, J6, J7: renamed from J?; footprint (none) -> Connector_PinSocket_2.54mm:PinSocket_1x03_P2.54mm_Vertical
- R1, R2, R3, R4: renamed from R?; footprint (none) -> Resistor_SMD:R_0603_1608Metric_Pad0.98x0.95mm_HandSolder
- RV1: renamed from RV?; value R_Potentiometer -> 10k; footprint (none) -> Potentiometer_THT:Potentiometer_Alpha_RD901F-40-00D_Single_Vertical
- SW1, SW2: renamed from SW?; footprint (none) -> Thonkiconn:Switch_Sub-Minitiature_Vertical
Connections:
- net +12V: now also J12.1 (Pin_1), J12.2 (Pin_2)
- net -12V: now also J12.5 (Pin_5), J12.6 (Pin_6)
- net GND: now also C3.2, C4.1, C1.2, C2.1, J12.3 (Pin_3), J12.4 (Pin_4)
- net at C3.1, D1.1 (K), F1.1: now also C1.1
- net at R1.2: now also J16.2 (Pin_2)
- net at C4.2, D2.2 (A), F2.1: now also C2.2
- net at R2.2: now also J13.2 (Pin_2)
- net at R3.2: now also J14.2 (Pin_2)
- net at R4.2: now also J15.2 (Pin_2)
- net at J1.1 (Pin_1), J1.2 (Pin_2): now also D2.1 (K); no longer D1.2 (A)
- net at J1.10 (Pin_10), J1.9 (Pin_9): now also D1.2 (A); no longer D2.1 (K)
- net at J11.TN: now also J15.1 (Pin_1)
- net at J9.TN: now also J13.1 (Pin_1)
- net at J10.TN: now also J14.1 (Pin_1)
- net at J8.TN: now also J16.1 (Pin_1)
- new net: J3.1 (Pin_1), RV2.1
- new net: J3.2 (Pin_2), RV2.2
- new net: J3.3 (Pin_3), RV2.3
- new net: J5.1 (Pin_1), RV4.1
- new net: J5.2 (Pin_2), RV4.2
- new net: J5.3 (Pin_3), RV4.3
- new net: J4.1 (Pin_1), RV3.1
- new net: J4.2 (Pin_2), RV3.2
- new net: J4.3 (Pin_3), RV3.3
Other:
- company: (none) -> L. Rittel
- moved on the sheet: C3, C4, D1, D2, F1, F2, J1, J10, J11, J2, J6, J7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

Commit message: breakout: finalize the pcb
Parts:
- J1: footprint Connector_PinSocket_2.54mm:PinSocket_2x05_P2.54mm_Vertical -> Connector_PinHeader_2.54mm:PinHeader_2x05_P2.54mm_Vertical
Changed lines of the file:
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@@
       (effects (font (size 1.27 1.27)) hide)
     )
-    (property "Footprint" "Connector_PinSocket_2.54mm:PinSocket_2x05_P2.54mm_Vertical" (id 2) (at 100.33 48.26 0)
+    (property "Footprint" "Connector_PinHeader_2.54mm:PinHeader_2x05_P2.54mm_Vertical" (id 2) (at 100.33 48.26 0)
       (effects (font (size 1.27 1.27)) hide)
     )
@@
     )
     (path "/94d0ad44-79f1-4cf2-b4c4-45fde72f1324"
-      (reference "J1") (unit 1) (value "Conn_02x05_Odd_Even") (footprint "Connector_PinSocket_2.54mm:PinSocket_2x05_P2.54mm_Vertical")
+      (reference "J1") (unit 1) (value "Conn_02x05_Odd_Even") (footprint "Connector_PinHeader_2.54mm:PinHeader_2x05_P2.54mm_Vertical")
     )
     (path "/740fb4bf-2e99-4976-b001-833aae14f32a"
