File: vco/frontpanel/vco_frontpanel.kicad_pcb (KiCad board)
At the start: 2 copper layers, 50.5 x 128.5 mm, 35 parts

Commit message: vco: Finished work on the front panel
Parts:
- removed SYM1: Circular_Scale, My_Misc:Pot_Scale_M7_300deg_0_10_d2.4
- removed SYM10, SYM11, SYM12, SYM13, SYM14: Jack_Marker_Output, My_Misc:Jack_Marker_Output
- removed SYM2, SYM3, SYM4, SYM5: Circular_Scale, My_Misc:Pot_Scale_M7_300deg_0_10_d2.0
- removed SYM6, SYM7, SYM8, SYM9: Jack_Marker_Input, My_Misc:Jack_Marker_Input
- added G***: LOGO, LOGO, F.Cu at (152.4, 96.7)
Routing:
- added copper zone on B.Cu, net (none)
- added copper zone on F.Cu, net (none)
Other:
- board text added: "JLCJLCJLCJLC"
- board text removed: "(VC|LF)O"
- board text removed: "1V/oct"
- board text removed: "Coarse"
- board text removed: "Exp"
- board text removed: "FM"
- board text removed: "FM Depth"
- board text removed: "Fine"
- board text removed: "LFO"
- board text removed: "Lin"
- board text removed: "PW"
- board text removed: "PW CV"
- board text removed: "Sync"
- board text removed: "VCO"

Commit message: vco: fix screw locations on the front panel
Parts:
- moved H4 35.6 mm to (170.1, 157.8)
- moved H3 35.5 mm to (134.5, 157.8)
- moved H12 0.19 mm to (173.9, 45.8)
- moved H2 0.06 mm to (170.1, 35.3)
Changed lines of the file:
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@@
     (pad "" np_thru_hole circle locked (at 0 0) (size 7.4 7.4) (drill 7.4) (layers F&B.Cu *.Mask))
   )
-  (footprint "MountingHole:MountingHole_3.2mm_M3" locked (layer "F.Cu")
-    (at 170 157.77)
+  (footprint "MountingHole:MountingHole_3.2mm_M3" (layer "F.Cu")
+    (at 134.5 157.77)
     (descr "Mounting Hole 3.2mm, no annular, M3")
     (tags "mounting hole 3.2mm no annular m3")
@@
     (fp_circle (center 0 0) (end 3.2 0) (layer "Cmts.User") (width 0.15) (fill none))
     (fp_circle (center 0 0) (end 3.45 0) (layer "F.CrtYd") (width 0.05) (fill none))
-    (pad "" np_thru_hole circle locked (at 0 0) (size 3.2 3.2) (drill 3.2) (layers *.Cu *.Mask))
+    (pad "" np_thru_hole circle (at 0 0) (size 3.2 3.2) (drill 3.2) (layers *.Cu *.Mask))
   )
   (footprint "MountingHole:MountingHole_6.4mm_M6" locked (layer "F.Cu")
@@
     (pad "" np_thru_hole circle locked (at 0 0) (size 6.4 6.4) (drill 6.4) (layers *.Cu *.Mask))
   )
-  (footprint "MountingHole:MountingHole_3.2mm_M3" locked (layer "F.Cu")
+  (footprint "MountingHole:MountingHole_3.2mm_M3" (layer "F.Cu")
     (at 134.5 35.27)
     (descr "Mounting Hole 3.2mm, no annular, M3")
@@
     (pad "" np_thru_hole circle locked (at 0 0) (size 3.2 3.2) (drill 3.2) (layers *.Cu *.Mask))
   )
-  (footprint "MountingHole:MountingHole_3.2mm_M3" locked (layer "F.Cu")
-    (at 134.5 157.77)
+  (footprint "MountingHole:MountingHole_3.2mm_M3" (layer "F.Cu")
+    (at 170.06 157.77)
     (descr "Mounting Hole 3.2mm, no annular, M3")
     (tags "mounting hole 3.2mm no annular m3")
@@
     (fp_circle (center 0 0) (end 3.2 0) (layer "Cmts.User") (width 0.15) (fill none))
     (fp_circle (center 0 0) (end 3.45 0) (layer "F.CrtYd") (width 0.05) (fill none))
-    (pad "" np_thru_hole circle locked (at 0 0) (size 3.2 3.2) (drill 3.2) (layers *.Cu *.Mask))
+    (pad "" np_thru_hole circle (at 0 0) (size 3.2 3.2) (drill 3.2) (layers *.Cu *.Mask))
   )
   (footprint "My_Misc:MountingHole_7.4mm_M7" locked (layer "F.Cu")
@@
   )
   (footprint "MountingHole:MountingHole_3.2mm_M3" locked (layer "F.Cu")
-    (at 173.75 45.6477)
+    (at 173.86 45.8)
     (descr "Mounting Hole 3.2mm, no annular, M3")
     (tags "mounting hole 3.2mm no annular m3")
@@
     (pad "" np_thru_hole circle locked (at 0 0) (size 5 5) (drill 5) (layers *.Cu *.Mask))
   )
-  (footprint "MountingHole:MountingHole_3.2mm_M3" locked (layer "F.Cu")
-    (at 170 35.27)
+  (footprint "MountingHole:MountingHole_3.2mm_M3" (layer "F.Cu")
+    (at 170.06 35.27)
     (descr "Mounting Hole 3.2mm, no annular, M3")
     (tags "mounting hole 3.2mm no annular m3")
