File: vco/frontpanel/vco_frontpanel.kicad_sch (KiCad schematic)
At the start: 35 parts

Commit message: vco: fix screw locations on the front panel
Parts:
- removed SYM1: Circular_Scale, My_Misc:Pot_Scale_M7_300deg_0_10_d2.4, symbol My_Misc:Circular_Scale
- removed SYM10, SYM11, SYM12, SYM13, SYM14: Jack_Marker_Output, My_Misc:Jack_Marker_Output, symbol My_Misc:Jack_Marker_Output
- removed SYM2, SYM3, SYM4, SYM5: Circular_Scale, My_Misc:Pot_Scale_M7_300deg_0_10_d2.0, symbol My_Misc:Circular_Scale
- removed SYM6, SYM7, SYM8, SYM9: Jack_Marker_Input, My_Misc:Jack_Marker_Input, symbol My_Misc:Jack_Marker_Input
